File: hardware/DWP 2020/DWP 2020.kicad_pcb (KiCad board)
At the start: 2 copper layers, 97.8 x 77.5 mm, 26 parts, among them K3 SNR03005, K4 SNR03005, T1 TIP32, T2 2SC1815

Commit message: Updated Kicad schematic
Other:
- board text added: "Hyperwiper V2.0.0"
- board text removed: "Dancing Wiper"
Changed lines of the file:
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@@
-(kicad_pcb (version 20200518) (host pcbnew "5.99.0-unknown-40250c4~88~ubuntu18.04.1")
+(kicad_pcb (version 20200518) (host pcbnew "5.99.0-unknown-6083c08~88~ubuntu18.04.1")
   (general
     (thickness 1.6)
@@
       (effects (font (size 1.27 1.27) (thickness 0.15)))
     )
-    (fp_text user " https://creativecommons.org/licenses/by-sa/3.0/" (at 0 -2.54) (layer "F.SilkS")
-      (effects (font (size 1.2065 1.2065) (thickness 0.1016)) (justify left bottom))
-    )
   )
   (module "TO-220-ALT" (layer "Top")
@@
   (gr_line (start 197.364661 68.8086) (end 197.364661 139.9286) (layer "Edge.Cuts") (width 0.4064))
   (gr_arc (start 194.189661 140.5636) (end 194.824661 143.7386) (angle -90) (layer "Edge.Cuts") (width 0.4064))
-  (gr_text "Dancing Wiper " (at 156.724661 80.2386) (layer "F.SilkS")
-    (effects (font (size 3.6195 3.6195) (thickness 0.3048)) (justify left bottom))
+  (gr_text "Hyperwiper\nV2.0.0" (at 178.308 137.414) (layer "F.SilkS")
+    (effects (font (size 2 2) (thickness 0.3048)) (justify left bottom))
   )
   (segment (start 118.599261 134.1628) (end 118.624661 134.2136) (width 0.762) (layer "Bottom") (net 32))

Commit message: Updated Kcad files
Parts:
- U$1: value TEENSY_3.1 -> TEENSY_4
Changed lines of the file:
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@@
-(kicad_pcb (version 20200518) (host pcbnew "5.99.0-unknown-6083c08~88~ubuntu18.04.1")
+(kicad_pcb (version 20200518) (host pcbnew "5.99.0-unknown-1973153~88~ubuntu18.04.1")
   (general
     (thickness 1.6)
@@
       (effects (font (size 1.2065 1.2065) (thickness 0.1016)) (justify left bottom))
     )
-    (fp_text value "TEENSY_3.1" (at -3.81 13.97) (layer "F.Fab")
+    (fp_text value "TEENSY_4" (at -3.81 13.97) (layer "F.Fab")
       (effects (font (size 1.2065 1.2065) (thickness 0.1016)) (justify left bottom))
     )
@@
     (pad "A11" thru_hole circle (at 5.08 -3.81) (size 1.4732 1.4732) (drill 0.9652) (layers *.Cu *.Mask)
       (solder_mask_margin 0.1016))
+    (model "/usr/share/kicad/modules/Teensy.pretty/Teensy_4.0_Assembly.STEP"
+      (offset (xyz 9.5 -32.5 -11.5))
+      (scale (xyz 1 1 1))
+      (rotate (xyz -90 0 90))
+    )
   )
   (module "AXIAL-0.3EZ" (layer "Top")

Commit message: fix some typoos
Parts:
- SSD1351: value SSD1351_128X128_LCD -> SSD1351_128X128; footprint SSD1351_128X128_LCD -> DWP2020 prototype:SSD1351_128X128_LCD
- moved SSD1351 0.26 mm to (172.1, 88.9)
Connections:
- SSD1351 pad JP1$1: D14 -> Net-(SSD1351-PadJP1$1)
- SSD1351 pad JP1$10: D10 -> /D10
- SSD1351 pad JP1$11: D12 -> Net-(SSD1351-PadJP1$11)
- SSD1351 pad JP1$2: D9 -> Net-(SSD1351-PadJP1$2)
- SSD1351 pad JP1$3: (no net) -> Net-(SSD1351-PadJP1$3)
- SSD1351 pad JP1$4: (no net) -> Net-(SSD1351-PadJP1$4)
- SSD1351 pad JP1$5: (no net) -> Net-(SSD1351-PadJP1$5)
- SSD1351 pad JP1$7: VCC -> /VCC
- SSD1351 pad JP1$9: D11 -> Net-(SSD1351-PadJP1$9)
