File: hardware/DWP 2020/DWP 2020.kicad_sch (KiCad schematic)
At the start: 22 parts, among them IC2 V_REG_78XX-TO-220, K3 SNR?0, K4 SNR?0, T1 TIP32, T2 2SC1815, X1 W237-3E, X2 W237-3E

Commit message: Updated Kicad schematic
Parts:
- removed FRAME1: FRAME-LETTER, bGeigieNanoKit V1.1r5a:CREATIVE_COMMONS, symbol import-from-eagle-rescue:FRAME-LETTER-bGeigieNanoKit_V1.1r5a-eagle-import
Other:
- company: (none) -> YR-Design/University of Aizu
- title: (none) -> Hyperwiper
Changed lines of the file:
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@@
-(kicad_sch (version 20200602) (host eeschema "5.99.0-unknown-40250c4~88~ubuntu18.04.1")
+(kicad_sch (version 20200602) (host eeschema "5.99.0-unknown-6083c08~88~ubuntu18.04.1")
   (page 1 1)
   (paper "User" 298.221 224.688)
+  (title_block
+    (title "Hyperwiper")
+    (date "2020-06-07")
+    (company "YR-Design/University of Aizu")
+  )
   (junction (at 41.91 137.16))
   (junction (at 64.77 157.48))
@@
     )
   )
-  (symbol (lib_id "import-from-eagle-rescue:FRAME-LETTER-bGeigieNanoKit_V1.1r5a-eagle-import") (at 175.26 203.2 0) (unit 2)
-    (in_bom yes)
-    (property "Reference" "FRAME1" (id 0) (at 175.26 203.2 0)
-      (effects (font (size 1.27 1.27)) hide)
-    )
-    (property "Value" "FRAME-LETTER" (id 1) (at 175.26 203.2 0)
-      (effects (font (size 1.27 1.27)) hide)
-    )
-    (property "Footprint" "bGeigieNanoKit V1.1r5a:CREATIVE_COMMONS" (id 2) (at 175.26 203.2 0)
-      (effects (font (size 1.27 1.27)) hide)
-    )
-    (property "Datasheet" "" (id 3) (at 175.26 203.2 0)
-      (effects (font (size 1.27 1.27)) hide)
-    )
-  )
   (symbol_instances
     (path "/469e1efe-1fe2-4e62-a629-b91661ee263e"
@@
       (reference "F1") (unit 1)
     )
-    (path "/f4fc1fc3-1446-4c9c-9172-bc3b85832d6c"
-      (reference "FRAME1") (unit 2)
-    )
     (path "/b29741e2-aef2-4043-8799-7b3ab7d17fa1"

Commit message: Updated Kcad files
Parts:
- U$1: value TEENSY_3.1 -> TEENSY_4
Changed lines of the file:
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@@
-(kicad_sch (version 20200602) (host eeschema "5.99.0-unknown-6083c08~88~ubuntu18.04.1")
+(kicad_sch (version 20200602) (host eeschema "5.99.0-unknown-2401ed5~88~ubuntu18.04.1")
   (page 1 1)
   (paper "User" 298.221 224.688)
@@
       (effects (font (size 1.27 1.27) bold) (justify left bottom))
     )
-    (property "Value" "TEENSY_3.1" (id 1) (at 112.014 106.68 0)
+    (property "Value" "TEENSY_4" (id 1) (at 112.014 106.68 0)
       (effects (font (size 1.27 1.27) bold) (justify left bottom))
     )

Commit message: fix some typoos
Parts:
- removed SSD1351: SSD1351_128X128_LCD, bGeigieNanoKit V1.1r5a:SSD1351_128X128_LCD, symbol import-from-eagle-rescue:SSD1351_128X128_LCD-bGeigieNanoKit_V1.1r5a-eagle-import
- added SSD1351: SSD1351_128X128, DWP2020 prototype:SSD1351_128X128_LCD, symbol import_from_eagle-rescue:SSD1351_128X128
- D2: symbol import-from-eagle-rescue:1N4004-bGeigieNanoKit_V1.1r5a-eagle-import -> Diode:1N4004
Connections:
- net 3.3V: now also SSD1351.JP1$6 (3.3V)
- net D10: now also SSD1351.JP1$10 (CL)
- net GND: now also SSD1351.JP1$8 (GND)
- net VCC: now also SSD1351.JP1$7 (VDD)
- net at IC2.IN, K3.14 (S), K3.A1 (1)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: now also D2.1 (K); no longer D2.C
- net at U$1.12: now also SSD1351.JP1$11 (DC)
- net at U$1.14/A0: now also SSD1351.JP1$1 (RST)
- net at U$1.9: now also SSD1351.JP1$9 (SI)
- net at K3.A2 (2), R2.P$1 (1): now also D2.2 (A); no longer D2.A
