File: hardware/DWP 2020/DWP 2020.kicad_sch (KiCad schematic)
At the start: 18 parts, among them IC2 V_REG_78XX-TO-220, K1 SNR?0-bGeigieNanoKit_V1.1r5a-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, K2 SNR?0-bGeigieNanoKit_V1.1r5a-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, T2 2SC1815, X1 W237-3E, X2 W237-3E

Commit message: Updated PCB
Parts:
- removed K1, K2: SNR?0-bGeigieNanoKit_V1.1r5a-eagle-import, DWP 2020:SNR-V, symbol import_from_eagle-rescue:SNR?0-bGeigieNanoKit_V1.1r5a-eagle-import
- removed SSD1351: SSD1351_128X128_LCD, SSD1351_128X128_LCD, symbol import-from-eagle-rescue:SSD1351_128X128_LCD-bGeigieNanoKit_V1.1r5a-eagle-import
- added K3, K4: SNR?0, bGeigieNanoKit V1.1r5a:SNR-V, symbol import-from-eagle-rescue:SNR?0-bGeigieNanoKit_V1.1r5a-eagle-import
- added R2: 33, bGeigieNanoKit V1.1r5a:AXIAL-0.5, symbol import-from-eagle-rescue:RESISTORPTH-1_2W-bGeigieNanoKit_V1.1r5a-eagle-import
- added R3: 1k, bGeigieNanoKit V1.1r5a:AXIAL-0.3EZ, symbol import-from-eagle-rescue:RESISTOREZ-bGeigieNanoKit_V1.1r5a-eagle-import
- added SSD1351: SSD1351_128X128, DWP2020 prototype:SSD1351_128X128_LCD, symbol import_from_eagle-rescue:SSD1351_128X128
- added T1: TIP32, bGeigieNanoKit V1.1r5a:TO220, symbol import-from-eagle-rescue:TIP32-bGeigieNanoKit_V1.1r5a-eagle-import
- D2: footprint DO41-10 -> bGeigieNanoKit V1.1r5a:DO41-10
- F1: footprint FUSE_HOLDER_5X20MM -> bGeigieNanoKit V1.1r5a:FUSE_HOLDER_5X20MM
- IC2: footprint TO-220-ALT -> bGeigieNanoKit V1.1r5a:TO-220-ALT
- JOYSWITCH1: footprint DWP 2020:SKQU -> bGeigieNanoKit V1.1r5a:SKQU
- LED1, LED2: footprint LED5MM -> bGeigieNanoKit V1.1r5a:LED5MM
- R1, R10, R4, R5: footprint AXIAL-0.3EZ -> bGeigieNanoKit V1.1r5a:AXIAL-0.3EZ
- S1: footprint CT10-A2 -> bGeigieNanoKit V1.1r5a:CT10-A2
- T2: footprint TO92-ECB -> bGeigieNanoKit V1.1r5a:TO92-ECB
- U$1: value TEENSY 4 -> TEENSY_4; footprint TEENSY_3.0+4 -> bGeigieNanoKit V1.1r5a:TEENSY_3.0+4
- X1, X2: footprint W237-3E -> bGeigieNanoKit V1.1r5a:W237-3E
Connections:
- net 3.3V: now also SSD1351.JP1$6 (3.3V)
- net D10: now also SSD1351.JP1$10 (CL)
- net GND: now also SSD1351.JP1$8 (GND), T1.2 (C)
- net VCC: now also SSD1351.JP1$7 (VDD)
- net at X1.1 (KL): now also K3.12 (O), K4.14 (S)
- net at X2.1 (KL): now also K4.A2 (2)
- net at F1.1: now also K3.11 (P), K4.A1 (1)
- net at D2.1 (K), IC2.IN: now also K3.14 (S), K3.A1 (1), K4.11 (P)
- net at T2.C: now also R3.P$1 (1); no longer D2.2 (A)
- net at U$1.12: now also SSD1351.JP1$11 (DC)
- net at U$1.14/A0: now also SSD1351.JP1$1 (RST)
- net at U$1.9: now also SSD1351.JP1$9 (SI)
- net A2): no longer names the net of U$1.16/A2
- net A3): no longer names the net of U$1.17/A3
- net A4): no longer names the net of U$1.18/A4
- net A5): no longer names the net of U$1.19/A5
- net A6): no longer names the net of U$1.20/A6
- net A7): no longer names the net of U$1.21/A7
- net A8): no longer names the net of U$1.22/A8
- net A9): no longer names the net of U$1.23/A9
- new net: R3.P$2 (2), T1.1 (B)
- new net: R2.P$2 (2), T1.3 (E)
- new net: D2.2 (A), K3.A2 (2), R2.P$1 (1)
Other:
- company: (none) -> YR-Design/University of Aizu
- title: (none) -> Hyperwiper
- moved on the sheet: R4, T2
