File: hardware/Hyperwiper 2020/Hyperwiper 2020.kicad_pcb (KiCad board)
At the start: 2 copper layers, 97.8 x 77.5 mm, 18 parts, among them IC2 V_REG_78XX-TO-220, K3 SNR-V, K4 SNR-V, T2 2SC1815, X1 W237-3E, X2 W237-3E

Commit message: Updated PCB
Parts:
- removed K3, K4: SNR-V, SNR-V
- added K1: SNR?0-bGeigieNanoKit_V1.1r5a-eagle-import, DWP 2020:SNR-V, F.Cu at (105.4, 113.0)
- added K2: SNR?0-bGeigieNanoKit_V1.1r5a-eagle-import, DWP 2020:SNR-V, F.Cu at (111.9, 113.0)
Connections:
- net Net-(U$1-Pad16/A2) renamed /A2)
- net Net-(U$1-Pad17/A3) renamed /A3)
- net Net-(U$1-Pad18/A4) renamed /A4)
- net Net-(U$1-Pad19/A5) renamed /A5)
- net Net-(U$1-Pad20/A6) renamed /A6)
- net Net-(U$1-Pad21/A7) renamed /A7)
- net Net-(U$1-Pad22/A8) renamed /A8)
- net Net-(U$1-Pad23/A9) renamed /A9)
Routing:
- net /D3: track 96.6 -> 108.5 mm
- net Net-(F1-Pad1): track 39.9 -> 29.7 mm
- net /VDD: track 121.1 -> 113.4 mm
- net Net-(K2-PadA2): track 26.5 -> 19.6 mm
- net /VCC: track 83.4 -> 89.7 mm
- net Net-(F1-Pad2): track 28.9 -> 31.3 mm
- net GND: track 233.9 -> 231.6 mm
- net /D4: track 105.9 -> 103.6 mm
- net Net-(D2-Pad1): track 78.3 -> 80.5 mm, vias 0 -> 1
- net /D8: track 150.4 -> 148.3 mm
- net /D2: track 106.2 -> 108.1 mm
- net Net-(D2-Pad2): track 51.7 -> 50.8 mm
- net Net-(LED2-PadA): track 26.3 -> 27.0 mm
