File: hardware/Hyperwiper 2020/Hyperwiper 2020 a.kicad_pcb (KiCad board)
At the start: 2 copper layers, 97.8 x 77.5 mm, 18 parts, among them IC2 V_REG_7805, K1 SONGLE SRA-12VDC-CL, K3 SONGLE SRA-12VDC-CL, T2 2SC1815, X1 W237-3E, X2 W237-3E

Commit message: Prototype production draft board.
Parts:
- moved S1 47.5 mm to (127.0, 125.7), turned to 180 degrees
- moved K3 37.3 mm to (74.8, 87.6), turned to 0 degrees
- moved F1 11.3 mm to (120.0, 118.1)
- moved K1 8.35 mm to (105.4, 113.0)
Connections:
- K1 pad 3: Net-(D2-Pad1) -> Net-(K1-Pad3)
- K1 pad 4: Net-(K1-Pad4) -> Net-(D2-Pad1)
- K3 pad 3: Net-(K1-Pad4) -> Net-(K1-Pad3)
- U$1 pad 5: /D5 -> Net-(U$1-Pad5)
- U$1 pad 6: /D6 -> Net-(U$1-Pad6)
- U$1 pad 7: /D7 -> Net-(U$1-Pad7)
- X1 pad 1: Net-(K1-Pad4) -> Net-(K1-Pad3)
Routing:
- net GND: track 222.3 -> 0.00 mm
- net /D8: track 142.5 -> 0.00 mm
- net /VDD: track 134.5 -> 0.00 mm
- net /D2: track 115.4 -> 0.00 mm
- net /D5: track 100.1 -> 0.00 mm
- net /D4: track 98.2 -> 0.00 mm
- net /D3: track 94.9 -> 0.00 mm
- net /VCC: track 89.4 -> 0.00 mm
- net Net-(D2-Pad2): track 86.9 -> 0.00 mm
- net /D7: track 81.9 -> 0.00 mm
- net Net-(SSD1351-PadJP1$2): track 78.0 -> 0.00 mm
- net /D6: track 76.2 -> 0.00 mm
- net Net-(SSD1351-PadJP1$11): track 76.2 -> 0.00 mm
- net Net-(D2-Pad1): track 73.0 -> 0.00 mm
- net Net-(K1-Pad4): track 70.6 -> 0.00 mm
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