File: hardware/Hyperwiper 2020/Hyperwiper 2020.kicad_sch (KiCad schematic)
At the start: 18 parts, among them IC2 V_REG_78XX-TO-220, K1 SNR?0-bGeigieNanoKit_V1.1r5a-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, K2 SNR?0-bGeigieNanoKit_V1.1r5a-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, T2 2SC1815, X1 W237-3E, X2 W237-3E

Commit message: Prototype production draft board.
Parts:
- removed K1, K2: SNR?0-bGeigieNanoKit_V1.1r5a-eagle-import, DWP 2020:SNR-V, symbol import_from_eagle-rescue:SNR?0-bGeigieNanoKit_V1.1r5a-eagle-import
- added K1, K3: SONGLE SRA-12VDC-CL, Relay_THT:Relay_SPDT_SANYOU_SRD_Series_Form_C, symbol Relay:SANYOU_SRD_Form_C
- D2: footprint DO41-10 -> Diode_THT:D_DO-41_SOD81_P10.16mm_Horizontal
- IC2: value V_REG_78XX-TO-220 -> V_REG_7805
- SSD1351: footprint SSD1351_128X128_LCD -> DWP2020 prototype:SSD1351_128X128_LCD
Connections:
- net D3 is gone; now on net VUSB: JOYSWITCH1.LEFT, JOYSWITCH1.UP, U$1.3
- net D5: now also U$1.5
- net D6: now also U$1.6
- net D7: now also U$1.7
- net VUSB: no longer U$1.VUSB
- net at X1.1 (KL): now also K1.4, K3.3
- net at X2.1 (KL): now also K1.5
- net at F1.1: now also K1.1, K1.2
- net at D2.1 (K), IC2.IN: now also K1.3, K3.1, K3.5
- net at D2.2 (A), T2.C: now also K3.2
Other:
- note removed: "notes: replace relay labeling K4 switch and K3 switches are revered.."
- moved on the sheet: D2
