File: hardware/Hyperwiper 2020 production prototype/_autosave-Hyperwiper 2020 production prototype.kicad_sch (KiCad schematic)
At the start: 19 parts, among them K1 Main Power relay, K2 Wiper control relay, Q1 PN2222A, SW1 ON-OFF, U1 Teensy4.0, U3 L7805

Commit message: Updated darft schemetics and board.
Parts:
- RV1: footprint Potentiometer_THT:Potentiometer_Alps_RK09K_Single_Horizontal -> Potentiometer_THT:Potentiometer_Piher_PT-10-V05_Vertical
- U3: footprint Package_TO_SOT_THT:TO-220-3_Vertical -> Package_TO_SOT_THT:TO-220-3_Horizontal_TabUp
Changed lines of the file:
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@@
   (symbol (lib_id "power:GND") (at 118.11 86.36 0) (unit 1)
     (in_bom yes) (on_board yes)
-    (property "Reference" "#PWR?" (id 0) (at 118.11 92.71 0)
+    (property "Reference" "#PWR0109" (id 0) (at 118.11 92.71 0)
       (effects (font (size 1.27 1.27)) hide)
     )
@@
       (effects (font (size 1.27 1.27)) (justify right))
     )
-    (property "Footprint" "Potentiometer_THT:Potentiometer_Alps_RK09K_Single_Horizontal" (id 2) (at 161.29 160.02 0)
+    (property "Footprint" "Potentiometer_THT:Potentiometer_Piher_PT-10-V05_Vertical" (id 2) (at 161.29 160.02 0)
       (effects (font (size 1.27 1.27)) hide)
     )
@@
     (property "Reference" "U3" (id 0) (at 241.3 21.59 0))
     (property "Value" "L7805" (id 1) (at 241.3 24.13 0))
-    (property "Footprint" "Package_TO_SOT_THT:TO-220-3_Vertical" (id 2) (at 241.935 33.02 0)
+    (property "Footprint" "Package_TO_SOT_THT:TO-220-3_Horizontal_TabUp" (id 2) (at 241.935 33.02 0)
       (effects (font (size 1.27 1.27) italic) (justify left) hide)
     )
@@
     )
     (path "/9b49453a-7d8c-46f7-ac72-5b7ca2259e26"
-      (reference "#PWR?") (unit 1)
+      (reference "#PWR0109") (unit 1)
     )
     (path "/3e7c7f71-990b-4b23-8faa-21bc92ed5e62"
