File: hardware/Hyperwiper 2020 production prototype/Hyperwiper 2020 production prototype.kicad_pcb (KiCad board)
At the start: 2 copper layers, 79.5 x 57.3 mm, 19 parts, among them K1 Main Power relay, K2 Wiper control relay, Q1 PN2222A, U1 Teensy4.0, U3 L7805, X1 W237-3E-bGeigieNanoKit_V1.1r5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, X2 W237-3E-bGeigieNanoKit_V1.1r5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

Commit message: Update Schematic and boards
Routing:
- net GND: track 0.00 -> 130.3 mm
- net /5V: track 0.00 -> 114.4 mm
- net Net-(Q1-Pad2): track 0.00 -> 57.7 mm
- net Net-(D2-Pad2): track 0.00 -> 52.2 mm
- net Net-(K1-Pad1): track 0.00 -> 51.8 mm
- net Net-(K1-Pad4): track 0.00 -> 51.7 mm
- net Net-(K2-Pad2): track 0.00 -> 45.6 mm
- net Net-(D3-Pad2): track 0.00 -> 38.1 mm
- net Net-(D1-Pad3): track 0.00 -> 37.4 mm
- net Net-(D2-Pad3): track 0.00 -> 35.3 mm
- net Net-(D1-Pad4): track 0.00 -> 34.8 mm
- net Net-(D2-Pad4): track 0.00 -> 31.5 mm
- net Net-(K1-Pad3): track 0.00 -> 25.6 mm
- net Net-(D1-Pad2): track 0.00 -> 23.6 mm
Changed lines of the file:
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@@
     (thickness 1.6)
     (drawings 8)
-    (tracks 0)
+    (tracks 102)
     (modules 19)
     (nets 16)
@@
   (gr_line (start 978.662 7.62) (end 978.662 62.357) (layer "Edge.Cuts") (width 0.05))
   (gr_line (start 900.43 6.35) (end 977.392 6.35) (layer "Edge.Cuts") (width 0.05))
+  (segment (start 912.188 15.598) (end 912.188 11.603) (width 0.25) (layer "B.Cu") (net 14))
+  (segment (start 926.211 29.621) (end 912.188 15.598) (width 0.25) (layer "B.Cu") (net 14))
+  (segment (start 926.211 36.195) (end 926.211 29.621) (width 0.25) (layer "B.Cu") (net 14))
+  (segment (start 931.806 41.79) (end 931.806 55.245) (width 0.25) (layer "B.Cu") (net 14))
+  (segment (start 926.211 36.195) (end 931.806 41.79) (width 0.25) (layer "B.Cu") (net 14))
+  (segment (start 975.945 16.46) (end 975.36 15.875) (width 0.25) (layer "B.Cu") (net 13))
+  (segment (start 975.945 51.485) (end 975.945 16.46) (width 0.25) (layer "B.Cu") (net 13))
+  (segment (start 974.344 53.086) (end 975.945 51.485) (width 0.25) (layer "B.Cu") (net 13))
+  (segment (start 975.539 24.571) (end 974.344 23.376) (width 0.25) (layer "F.Cu") (net 12))
+  (segment (start 975.539 37.883) (end 975.539 24.571) (width 0.25) (layer "F.Cu") (net 12))
+  (segment (start 963.785 49.637) (end 975.539 37.883) (width 0.25) (layer "F.Cu") (net 12))
+  (segment (start 952.027 49.637) (end 963.785 49.637) (width 0.25) (layer "F.Cu") (net 12))
+  (segment (start 948.324 53.34) (end 952.027 49.637) (width 0.25) (layer "F.Cu") (net 12))
+  (segment (start 945.896 53.34) (end 948.324 53.34) (width 0.25) (layer "F.Cu") (net 12))
+  (segment (start 974.344 22.25) (end 974.344 23.376) (width 0.25) (layer "F.Cu") (net 12))
+  (segment (start 962.559 46.219) (end 973.218 35.56) (width 0.25) (layer "F.Cu") (net 11))
+  (segment (start 954.611 46.219) (end 962.559 46.219) (width 0.25) (layer "F.Cu") (net 11))
+  (segment (start 948.76 52.07) (end 954.611 46.219) (width 0.25) (layer "F.Cu") (net 11))
+  (segment (start 945.896 52.07) (end 948.76 52.07) (width 0.25) (layer "F.Cu") (net 11))
+  (segment (start 974.344 35.56) (end 973.218 35.56) (width 0.25) (layer "F.Cu") (net 11))
+  (segment (start 964.088 40.64) (end 969.168 35.56) (width 0.25) (layer "F.Cu") (net 10))
+  (segment (start 956.509 40.64) (end 964.088 40.64) (width 0.25) (layer "F.Cu") (net 10))
+  (segment (start 953.516 43.633) (end 956.509 40.64) (width 0.25) (layer "F.Cu") (net 10))
+  (segment (start 953.516 45.061) (end 953.516 43.633) (width 0.25) (layer "F.Cu") (net 10))
+  (segment (start 947.777 50.8) (end 953.516 45.061) (width 0.25) (layer "F.Cu") (net 10))
+  (segment (start 945.896 50.8) (end 947.777 50.8) (width 0.25) (layer "F.Cu") (net 10))
+  (segment (start 970.294 35.56) (end 969.168 35.56) (width 0.25) (layer "F.Cu") (net 10))
+  (segment (start 953.77 53.34) (end 954.996 53.34) (width 0.25) (layer "B.Cu") (net 9))
+  (segment (start 966.089 42.247) (end 954.996 53.34) (width 0.25) (layer "B.Cu") (net 9))
+  (segment (start 966.089 35.56) (end 966.089 42.247) (width 0.25) (layer "B.Cu") (net 9))
+  (segment (start 964.185 29.485) (end 970.294 23.376) (width 0.25) (layer "B.Cu") (net 8))
+  (segment (start 964.185 42.881) (end 964.185 29.485) (width 0.25) (layer "B.Cu") (net 8))
+  (segment (start 954.996 52.07) (end 964.185 42.881) (width 0.25) (layer "B.Cu") (net 8))
+  (segment (start 953.77 52.07) (end 954.996 52.07) (width 0.25) (layer "B.Cu") (net 8))
+  (segment (start 970.294 22.25) (end 970.294 23.376) (width 0.25) (layer "B.Cu") (net 8))
+  (segment (start 953.77 50.8) (end 954.996 50.8) (width 0.25) (layer "B.Cu") (net 7))
+  (segment (start 966.089 22.25) (end 966.089 23.376) (width 0.25) (layer "B.Cu") (net 7))
+  (segment (start 956.056 49.74) (end 954.996 50.8) (width 0.25) (layer "B.Cu") (net 7))
+  (segment (start 956.056 44.066) (end 956.056 49.74) (width 0.25) (layer "B.Cu") (net 7))
+  (segment (start 959.482 40.64) (end 956.056 44.066) (width 0.25) (layer "B.Cu") (net 7))
+  (segment (start 960.238 40.64) (end 959.482 40.64) (width 0.25) (layer "B.Cu") (net 7))
+  (segment (start 962.427 38.451) (end 960.238 40.64) (width 0.25) (layer "B.Cu") (net 7))
+  (segment (start 962.427 27.038) (end 962.427 38.451) (width 0.25) (layer "B.Cu") (net 7))
+  (segment (start 966.089 23.376) (end 962.427 27.038) (width 0.25) (layer "B.Cu") (net 7))
+  (segment (start 974.205 11.43) (end 975.36 11.43) (width 0.25) (layer "F.Cu") (net 6))
+  (segment (start 960.235 25.4) (end 974.205 11.43) (width 0.25) (layer "F.Cu") (net 6))
+  (segment (start 959.482 25.4) (end 960.235 25.4) (width 0.25) (layer "F.Cu") (net 6))
+  (segment (start 948.436 36.446) (end 959.482 25.4) (width 0.25) (layer "F.Cu") (net 6))
+  (segment (start 948.436 41.54) (end 948.436 36.446) (width 0.25) (layer "F.Cu") (net 6))
+  (segment (start 945.896 44.08) (end 948.436 41.54) (width 0.25) (layer "F.Cu") (net 6))
+  (segment (start 945.896 45.354) (end 945.896 44.08) (width 0.25) (layer "F.Cu") (net 6))
+  (segment (start 940.51 50.74) (end 945.896 45.354) (width 0.25) (layer "F.Cu") (net 6))
+  (segment (start 938.784 50.74) (end 940.51 50.74) (width 0.25) (layer "F.Cu") (net 6))
+  (segment (start 938.784 51.816) (end 938.784 50.74) (width 0.25) (layer "F.Cu") (net 6))
+  (segment (start 967.53 56.134) (end 960.628 56.134) (width 0.25) (layer "F.Cu") (net 5))
+  (segment (start 970.578 53.086) (end 967.53 56.134) (width 0.25) (layer "F.Cu") (net 5))
+  (segment (start 971.804 53.086) (end 970.578 53.086) (width 0.25) (layer "F.Cu") (net 5))
+  (segment (start 940.054 51.816) (end 940.054 52.892) (width 0.25) (layer "F.Cu") (net 5))
+  (segment (start 915.416 55.245) (end 916.637 55.245) (width 0.25) (layer "F.Cu") (net 5))
+  (segment (start 956.52 56.134) (end 960.628 56.134) (width 0.25) (layer "F.Cu") (net 5))
+  (segment (start 954.996 54.61) (end 956.52 56.134) (width 0.25) (layer "F.Cu") (net 5))
+  (segment (start 953.77 54.61) (end 954.996 54.61) (width 0.25) (layer "F.Cu") (net 5))
+  (segment (start 907.49 37.032) (end 903.986 33.528) (width 0.25) (layer "F.Cu") (net 5))
+  (segment (start 907.49 41.392) (end 907.49 37.032) (width 0.25) (layer "F.Cu") (net 5))
+  (segment (start 918.99 52.892) (end 907.49 41.392) (width 0.25) (layer "F.Cu") (net 5))
+  (segment (start 918.99 52.892) (end 916.637 55.245) (width 0.25) (layer "F.Cu") (net 5))
+  (segment (start 940.054 52.892) (end 918.99 52.892) (width 0.25) (layer "F.Cu") (net 5))
+  (segment (start 941.772 54.61) (end 945.896 54.61) (width 0.25) (layer "F.Cu") (net 5))
+  (segment (start 940.054 52.892) (end 941.772 54.61) (width 0.25) (layer "F.Cu") (net 5))
+  (segment (start 952.544 47.923) (end 952.544 54.61) (width 0.25) (layer "B.Cu") (net 5))
+  (segment (start 953.659 46.808) (end 952.544 47.923) (width 0.25) (layer "B.Cu") (net 5))
+  (segment (start 953.659 20.177) (end 953.659 46.808) (width 0.25) (layer "B.Cu") (net 5))
+  (segment (start 959.866 13.97) (end 953.659 20.177) (width 0.25) (layer "B.Cu") (net 5))
+  (segment (start 953.77 54.61) (end 952.544 54.61) (width 0.25) (layer "B.Cu") (net 5))
+  (segment (start 945.896 54.61) (end 952.544 54.61) (width 0.25) (layer "B.Cu") (net 5))
+  (segment (start 937.514 24.729) (end 937.514 51.816) (width 0.25) (layer "B.Cu") (net 4))
+  (segment (start 924.388 11.603) (end 937.514 24.729) (width 0.25) (layer "B.Cu") (net 4))
+  (segment (start 906.138 36.068) (end 903.986 36.068) (width 0.25) (layer "B.Cu") (net 3))
+  (segment (start 912.061 30.145) (end 906.138 36.068) (width 0.25) (layer "B.Cu") (net 3))
+  (segment (start 917.846 30.145) (end 912.061 30.145) (width 0.25) (layer "F.Cu") (net 3))
+  (segment (start 924.388 23.603) (end 917.846 30.145) (width 0.25) (layer "F.Cu") (net 3))
+  (segment (start 926.726 44.61) (end 924.261 42.145) (width 0.25) (layer "B.Cu") (net 2))
+  (segment (start 926.726 55.245) (end 926.726 44.61) (width 0.25) (layer "B.Cu") (net 2))
+  (segment (start 924.211 42.195) (end 924.261 42.145) (width 0.25) (layer "F.Cu") (net 2))
+  (segment (start 912.011 42.195) (end 924.211 42.195) (width 0.25) (layer "F.Cu") (net 2))
+  (segment (start 926.338 30.837) (end 926.338 17.653) (width 0.25) (layer "F.Cu") (net 2))
+  (segment (start 924.261 32.914) (end 926.338 30.837) (width 0.25) (layer "F.Cu") (net 2))
+  (segment (start 924.261 42.145) (end 924.261 32.914) (width 0.25) (layer "F.Cu") (net 2))
+  (segment (start 908.635 30.988) (end 903.986 30.988) (width 0.25) (layer "F.Cu") (net 1))
+  (segment (start 926.924 12.699) (end 908.635 30.988) (width 0.25) (layer "F.Cu") (net 1))
+  (segment (start 958.597 12.699) (end 926.924 12.699) (width 0.25) (layer "F.Cu") (net 1))
+  (segment (start 959.866 11.43) (end 958.597 12.699) (width 0.25) (layer "F.Cu") (net 1))
+  (segment (start 965.2 15.875) (end 966.326 15.875) (width 0.25) (layer "B.Cu") (net 1))
+  (segment (start 971.636 21.185) (end 966.326 15.875) (width 0.25) (layer "B.Cu") (net 1))
+  (segment (start 971.636 22.673) (end 971.636 21.185) (width 0.25) (layer "B.Cu") (net 1))
+  (segment (start 968.643 25.666) (end 971.636 22.673) (width 0.25) (layer "B.Cu") (net 1))
+  (segment (start 968.643 40.725) (end 968.643 25.666) (width 0.25) (layer "B.Cu") (net 1))
+  (segment (start 960.628 48.74) (end 968.643 40.725) (width 0.25) (layer "B.Cu") (net 1))
+  (segment (start 960.628 51.134) (end 960.628 48.74) (width 0.25) (layer "B.Cu") (net 1))
+  (segment (start 964.074 15.638) (end 964.074 15.875) (width 0.25) (layer "B.Cu") (net 1))
+  (segment (start 959.866 11.43) (end 964.074 15.638) (width 0.25) (layer "B.Cu") (net 1))
+  (segment (start 965.2 15.875) (end 964.074 15.875) (width 0.25) (layer "B.Cu") (net 1))
 )
