File: hardware/Hyperwiper 2020 production prototype/Hyperwiper 2020 production prototype.kicad_pcb (KiCad board)
At the start: 2 copper layers, 123.8 x 65.8 mm, 22 parts, among them J1 Conn_01x05, J2 USB_B, Q2 2N3904, Q3 IRF4905, SW1 SW_DPDT_x2, SW2 SW_Reed, U1 Teensy4.0, U3 Voltage regulator

Commit message: Updates board
Parts:
- removed Q3: IRF4905, Package_TO_SOT_THT:TO-220-3_Vertical
- added C4: 100uf, Capacitor_THT:CP_Radial_D5.0mm_P2.50mm, F.Cu at (173.2, 92.6)
- added D5: 1n4001, Diode_THT:D_DO-35_SOD27_P10.16mm_Horizontal, F.Cu at (171.1, 100.1)
- added Q1: IRF3205, Package_TO_SOT_THT:TO-220-3_Vertical, F.Cu at (162.3, 82.9)
- R10, R2: value 10k -> 1k
- moved R10 73.2 mm to (108.6, 113.3)
- moved R2 73.2 mm to (98.4, 116.9)
- moved C1 26.9 mm to (185.4, 92.8), turned to 90 degrees
- moved SW1 21.7 mm to (186.3, 110.7)
- moved Q2 13.6 mm to (156.1, 112.1)
- moved C3 6.37 mm to (114.0, 115.8)
- moved RV1 4.38 mm to (160.8, 98.6)
Connections:
- D4 pad 2: (no net) -> Net-(D4-Pad2)
- J1 pad 1: Net-(J1-Pad1) -> Net-(D5-Pad1)
- R10 pad 2: Net-(J1-Pad1) -> Net-(C4-Pad1)
- RLY1 pad 1: Net-(J1-Pad1) -> Net-(D5-Pad1)
- RLY1 pad 5: (no net) -> Net-(D4-Pad2)
- SW1 pad 5: Net-(J1-Pad1) -> Net-(D5-Pad1)
- SW1 pad 6: (no net) -> Net-(D4-Pad2)
- U3 pad 1: (no net) -> Net-(D4-Pad2)
Routing:
- net /reed: track 151.5 -> 0.00 mm
- net /5V: track 104.5 -> 0.00 mm
- net +3V3: track 101.0 -> 0.00 mm
- net Net-(J2-Pad1): track 98.8 -> 0.00 mm
- net /motor_PWM: track 96.8 -> 0.00 mm
- net Net-(C4-Pad2): track 94.8 -> 0.00 mm
- net /M_LED_b: track 84.3 -> 0.00 mm
- net Net-(J1-Pad1): track 78.0 -> 0.00 mm
- net /M_LED_g: track 75.7 -> 0.00 mm
- net /Pot: track 75.1 -> 0.00 mm
- net /B_LED_b: track 74.6 -> 0.00 mm
- net /M_LED_r: track 72.6 -> 0.00 mm
- net TX-1: track 68.7 -> 0.00 mm
- net /B_LED_g: track 64.9 -> 0.00 mm
- net RX-1: track 63.1 -> 0.00 mm
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Other:
- board text added: "HyperWiper Prototype V2.4.1"
- board text removed: "HyperWiper Prototype V2.4.0"
