File: hardware/Hyperwiper 2020 production prototype/Hyperwiper 2020 production prototype.kicad_sch (KiCad schematic)
At the start: 27 parts, among them J1 Conn_01x05, Q2 2N3904, Q3 IRF4905, SW1 SW_DPDT_x2, SW2 SW_Reed, U1 Teensy4.0, U3 Voltage regulator

Commit message: Updated board for new layout
Parts:
- SW1: footprint (none) -> Button_Switch_THT:SW_CuK_JS202011CQN_DPDT_Straight
Changed lines of the file:
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@@
     (title "Prototype board")
     (date "2020-08-19")
-    (rev "V2.1.6")
+    (rev "V2.2.6")
   )
   (junction (at 127.635 88.9) (diameter 0.259) (color 0 0 0 0))
@@
   (symbol (lib_id "power:+3V3") (at 127.635 88.9 270) (unit 1)
     (in_bom yes) (on_board yes)
-    (property "Reference" "#PWR?" (id 0) (at 123.825 88.9 0)
+    (property "Reference" "#PWR0113" (id 0) (at 123.825 88.9 0)
       (effects (font (size 1.27 1.27)) hide)
     )
@@
   (symbol (lib_id "power:GND") (at 127.635 99.695 0) (unit 1)
     (in_bom yes) (on_board yes)
-    (property "Reference" "#PWR?" (id 0) (at 127.635 106.045 0)
+    (property "Reference" "#PWR0103" (id 0) (at 127.635 106.045 0)
       (effects (font (size 1.27 1.27)) hide)
     )
@@
       (effects (font (size 1.27 1.27)) (justify right))
     )
-    (property "Footprint" "" (id 2) (at 245.745 92.075 0)
+    (property "Footprint" "Button_Switch_THT:SW_CuK_JS202011CQN_DPDT_Straight" (id 2) (at 245.745 92.075 0)
       (effects (font (size 1.27 1.27)) hide)
     )
@@
       (effects (font (size 1.27 1.27)) (justify right))
     )
-    (property "Footprint" "" (id 2) (at 247.65 57.15 0)
+    (property "Footprint" "Button_Switch_THT:SW_CuK_JS202011CQN_DPDT_Straight" (id 2) (at 247.65 57.15 0)
       (effects (font (size 1.27 1.27)) hide)
     )
@@
       (reference "#PWR0102") (unit 1) (value "GND") (footprint "")
     )
+    (path "/10c7def5-12ac-453c-9a34-a49b0704d7bd"
+      (reference "#PWR0103") (unit 1) (value "GND") (footprint "")
+    )
     (path "/dc0b0cf5-d714-43fd-906e-7e8ba2bf804e"
       (reference "#PWR0104") (unit 1) (value "GND") (footprint "")
@@
       (reference "#PWR0112") (unit 1) (value "+3V3") (footprint "")
     )
+    (path "/babc2518-5094-496e-9bdc-d94851cfa9c2"
+      (reference "#PWR0113") (unit 1) (value "+3V3") (footprint "")
+    )
     (path "/46d8eafb-00fd-4bdf-87b9-dd5898c2f937"
       (reference "#PWR0114") (unit 1) (value "GND") (footprint "")
@@
       (reference "#PWR0116") (unit 1) (value "+3V3") (footprint "")
     )
-    (path "/10c7def5-12ac-453c-9a34-a49b0704d7bd"
-      (reference "#PWR?") (unit 1) (value "GND") (footprint "")
-    )
-    (path "/babc2518-5094-496e-9bdc-d94851cfa9c2"
-      (reference "#PWR?") (unit 1) (value "+3V3") (footprint "")
-    )
     (path "/bc80e3ce-b48d-40fd-b22c-6384e7899540"
       (reference "C1") (unit 1) (value "0.1uF") (footprint "Capacitor_THT:C_Rect_L7.0mm_W2.5mm_P5.00mm")
@@
     )
     (path "/708522b5-f48c-473c-8635-21f9ec15887b"
-      (reference "SW1") (unit 1) (value "SW_DPDT_x2") (footprint "")
+      (reference "SW1") (unit 1) (value "SW_DPDT_x2") (footprint "Button_Switch_THT:SW_CuK_JS202011CQN_DPDT_Straight")
     )
     (path "/06382058-0dbb-497c-b69a-5fa0882a27c2"
-      (reference "SW1") (unit 2) (value "SW_DPDT_x2") (footprint "")
+      (reference "SW1") (unit 2) (value "SW_DPDT_x2") (footprint "Button_Switch_THT:SW_CuK_JS202011CQN_DPDT_Straight")
     )
     (path "/dbeb2dea-7d69-49c5-950e-aaa8e36682a0"
