File: hardware/test/test/test.kicad_sch (KiCad schematic)
At the start: 0 parts

Commit message: Test for N-ch MOSFET 100A high end
Parts:
- added BT1: 12V, symbol Device:Battery_Cell
- added C1: 01.uF, symbol OPL_Capacitor:TANTALUM-SMD-10UF-10V-10%_AVX-A_
- added D1: DIODE, symbol Simulation_SPICE:DIODE
- added LA1: Lamp, symbol Device:Lamp
- added Q1: PN2222A, Package_TO_SOT_THT:TO-92_Inline, symbol Transistor_BJT:PN2222A
- added Q2: N-ch MOSFET, Package_TO_SOT_THT:TO-220-3_Vertical, symbol Transistor_FET:IPP060N06N
- added R1: 1K, symbol Device:R
- added R?: 10k, symbol Device:R
Connections:
- new net: BT1.1 (+), D1.1 (A), Q2.2 (D)
- new net: C1.1 (+), D1.2 (K), R1.1
- new net: Q1.3 (C), Q2.1 (G), R1.2
- new net: BT1.2 (-), LA1.1 (-), Q1.1 (E)
- new net: Q1.2 (B), R?.2
- new net: C1.2 (-), LA1.2 (+), Q2.3 (S)
Other:
- note added: "d"
- note added: "g"
- note added: "https://www.re-innovation.co.uk/docs/open-charge-regulator/charge-controller-project-power-switching/"
- note added: "s"
